Commit message: Updated robot_core for robot actual dimensions

File: description/robot_core.xacro (robot description, xacro)
@@ -22,22 +22,22 @@
         <parent link="base_link"/>
         <child link="chassis"/>
-        <origin xyz="-0.1 0 0"/>
+        <origin xyz="0 0 0"/>
     </joint>
     <link name="chassis">
         <visual>
-            <origin xyz="0.15 0 0.075"/>
+            <origin xyz="0 0 0.0455"/>
             <geometry>
-                <box size="0.3 0.3 0.15"/>
+                <box size="0.186 0.093 0.091"/>
             </geometry>
             <material name="white"/>
         </visual>
         <collision>
-            <origin xyz="0.15 0 0.075"/>
+            <origin xyz="0 0 0.0455"/>
             <geometry>
-                <box size="0.3 0.3 0.15"/>
+                <box size="0.186 0.093 0.091"/>
             </geometry>
         </collision>
-        <xacro:inertial_box mass="0.5" x="0.3" y="0.3" z="0.15">
-            <origin xyz="0.15 0 0.075" rpy="0 0 0"/>
+        <xacro:inertial_box mass="0.55" x="0.186" y="0.093" z="0.091">
+            <origin xyz="0 0 0.0455" rpy="0 0 0"/>
         </xacro:inertial_box>
     </link>
@@ -46,5 +46,5 @@
         <parent link="base_link"/>
         <child link="left_front_wheel"/>
-        <origin xyz="0.15 0.175 0" rpy="-${pi/2} 0 0"/>
+        <origin xyz="0.0676 0.0566 0" rpy="-${pi/2} 0 0"/>
         <axis xyz="0 0 1"/>
     </joint>
@@ -52,5 +52,5 @@
         <visual>
             <geometry>
-                <cylinder radius="0.05" length="0.04"/>
+                <cylinder radius="0.0325" length="0.02"/>
             </geometry>
             <material name="blue"/>
@@ -58,8 +58,8 @@
         <collision>
             <geometry>
-                <cylinder radius="0.05" length="0.04"/>
+                <cylinder radius="0.0325" length="0.02"/>
             </geometry>
         </collision>
-        <xacro:inertial_cylinder mass="0.1" length="0.04" radius="0.05">
+        <xacro:inertial_cylinder mass="0.0375" length="0.02" radius="0.0325">
             <origin xyz="0 0 0" rpy="0 0 0"/>
         </xacro:inertial_cylinder>
@@ -69,5 +69,5 @@
         <parent link="base_link"/>
         <child link="right_front_wheel"/>
-        <origin xyz="0.15 -0.175 0" rpy="${pi/2} 0 0"/>
+        <origin xyz="0.0676 -0.0566 0" rpy="${pi/2} 0 0"/>
         <axis xyz="0 0 -1"/>
     </joint>
@@ -75,5 +75,5 @@
         <visual>
             <geometry>
-                <cylinder radius="0.05" length="0.04"/>
+                <cylinder radius="0.0325" length="0.02"/>
             </geometry>
             <material name="blue"/>
@@ -81,8 +81,8 @@
         <collision>
             <geometry>
-                <cylinder radius="0.05" length="0.04"/>
+                <cylinder radius="0.0325" length="0.02"/>
             </geometry>
         </collision>
-        <xacro:inertial_cylinder mass="0.1" length="0.04" radius="0.05">
+        <xacro:inertial_cylinder mass="0.0375" length="0.02" radius="0.0325">
             <origin xyz="0 0 0" rpy="0 0 0"/>
         </xacro:inertial_cylinder>
@@ -92,5 +92,5 @@
         <parent link="base_link"/>
         <child link="left_rear_wheel"/>
-        <origin xyz="-0.05 0.175 0" rpy="-${pi/2} 0 0"/>
+        <origin xyz="-0.0676 0.0566 0" rpy="-${pi/2} 0 0"/>
         <axis xyz="0 0 1"/>
     </joint>
@@ -98,5 +98,5 @@
         <visual>
             <geometry>
-                <cylinder radius="0.05" length="0.04"/>
+                <cylinder radius="0.0325" length="0.02"/>
             </geometry>
             <material name="black"/>
@@ -104,8 +104,8 @@
         <collision>
             <geometry>
-                <cylinder radius="0.05" length="0.04"/>
+                <cylinder radius="0.0325" length="0.02"/>
             </geometry>
         </collision>
-        <xacro:inertial_cylinder mass="0.1" length="0.04" radius="0.05">
+        <xacro:inertial_cylinder mass="0.0375" length="0.02" radius="0.0325">
             <origin xyz="0 0 0" rpy="0 0 0"/>
         </xacro:inertial_cylinder>
@@ -115,5 +115,5 @@
         <parent link="base_link"/>
         <child link="right_rear_wheel"/>
-        <origin xyz="-0.05 -0.175 0" rpy="${pi/2} 0 0"/>
+        <origin xyz="-0.0676 -0.0566 0" rpy="${pi/2} 0 0"/>
         <axis xyz="0 0 -1"/>
     </joint>
@@ -121,5 +121,5 @@
         <visual>
             <geometry>
-                <cylinder radius="0.05" length="0.04"/>
+                <cylinder radius="0.0325" length="0.02"/>
             </geometry>
             <material name="black"/>
@@ -127,8 +127,8 @@
         <collision>
             <geometry>
-                <cylinder radius="0.05" length="0.04"/>
+                <cylinder radius="0.0325" length="0.02"/>
             </geometry>
         </collision>
-        <xacro:inertial_cylinder mass="0.1" length="0.04" radius="0.05">
+        <xacro:inertial_cylinder mass="0.0375" length="0.02" radius="0.0325">
             <origin xyz="0 0 0" rpy="0 0 0"/>
         </xacro:inertial_cylinder>
