Commit message: Created gazebo control

File: description/gazebo_control.xacro (robot description, xacro)
@@ -2,21 +2,26 @@
 <robot xmlns:xacro="http://www.ros.org/wiki/xacro">
     <gazebo>
-        <plugin name="diff_drive" filename="libgazebo_ros_diff_drive.so">
+        <plugin name="skid_steer_drive" filename="libgazebo_ros_diff_drive.so">
+            <ros>
+                <namespace> </namespace>
+            </ros>
             <!-- WHEEL INFORMATION -->
+             <num_wheel_pairs>2</num_wheel_pairs>
             <left_joint>left_front_wheel_joint</left_joint>
             <left_joint>left_rear_wheel_joint</left_joint>
             <right_joint>right_front_wheel_joint</right_joint>
             <right_joint>right_rear_wheel_joint</right_joint>
-            <wheel_separation>0.35</wheel_separation>
-            <wheel_diameter>0.1</wheel_diameter>
-            <!-- LIMITS -->
-            <max_wheel_torque>200</max_wheel_torque>
-            <max_wheel_acceleration>10.0</max_wheel_acceleration>
+            <wheel_separation>${wheel_separation}</wheel_separation>
+            <wheel_separation>${wheel_separation}</wheel_separation>
+            <wheel_diameter>${wheel_diameter}</wheel_diameter>
+            <wheel_diameter>${wheel_diameter}</wheel_diameter>
+            <max_wheel_torque>${gazebo_max_wheel_torque}</max_wheel_torque>
+            <max_wheel_acceleration>${gazebo_max_wheel_acceleration}</max_wheel_acceleration>
             <!-- OUTPUT -->
-            <odometry_frame>odom</odometry_frame>
-            <robot_base_frame>base_link</robot_base_frame>
             <publish_odom>true</publish_odom>
             <publish_odom_tf>true</publish_odom_tf>
             <publish_wheel_tf>true</publish_wheel_tf>
+            <odometry_frame>odom</odometry_frame>
+            <robot_base_frame>base_link</robot_base_frame>
         </plugin>
     </gazebo>

File: description/inertial_macros.xacro (robot description, xacro)
@@ -3,4 +3,7 @@
     <!-- Specify some standard inertial calculations https://en.wikipedia.org/wiki/List_of_moments_of_inertia -->
     <!-- These make use of xacro's mathematical functionality -->
+    <xacro:property name="chassis_x_dim" value="0.186"/>
+    <xacro:property name="chassis_y_dim" value="0.093"/>
+    <xacro:property name="chassis_z_dim" value="0.093"/>
     <xacro:macro name="inertial_box" params="mass x y z *origin">
         <inertial>

File: description/robot_core.xacro (robot description, xacro)
@@ -2,20 +2,7 @@
 <robot xmlns:xacro="http://www.ros.org/wiki/xacro" >
     <xacro:include filename="inertial_macros.xacro"/>
-    <!-- COLORS -->
-    <material name="white">
-        <color rgba="1 1 1 1"/>
-    </material>
-    <material name="orange">
-        <color rgba="1 0.3 0.1 1"/>
-    </material>
-    <material name="blue">
-        <color rgba="0.2 0.2 1 1"/>
-    </material>
-    <material name="black">
-        <color rgba="0 0 0 1"/>
-    </material>
+    <xacro:include filename="robot_params.xacro"/>
     <!-- BASE LINK -->
-    <link name="base_link">
-    </link>
+    <link name="base_link"/>
     <!-- CHASSIS -->
     <joint name="chassis_joint" type="fixed">
@@ -26,17 +13,17 @@
     <link name="chassis">
         <visual>
-            <origin xyz="0 0 0.0455"/>
+            <origin xyz="${chassis_origin_x} ${chassis_origin_y} ${chassis_origin_z}"/>
             <geometry>
-                <box size="0.186 0.093 0.091"/>
+                <box size="${chassis_length} ${chassis_width} ${chassis_height}"/>
             </geometry>
             <material name="white"/>
         </visual>
         <collision>
-            <origin xyz="0 0 0.0455"/>
+            <origin xyz="${chassis_origin_x} ${chassis_origin_y} ${chassis_origin_z}"/>
             <geometry>
-                <box size="0.186 0.093 0.091"/>
+                <box size="${chassis_length} ${chassis_width} ${chassis_height}"/>
             </geometry>
         </collision>
-        <xacro:inertial_box mass="0.55" x="0.186" y="0.093" z="0.091">
+        <xacro:inertial_box mass="${chassis_mass}" x="${chassis_length}" y="${chassis_width}" z="${chassis_height}">
             <origin xyz="0 0 0.0455" rpy="0 0 0"/>
         </xacro:inertial_box>
@@ -46,11 +33,13 @@
         <parent link="base_link"/>
         <child link="left_front_wheel"/>
-        <origin xyz="0.0676 0.0566 0" rpy="-${pi/2} 0 0"/>
+        <origin xyz="${wheel_x_offset} ${wheel_y_offset} ${wheel_z_offset}" rpy="-${pi/2} 0 0"/>
         <axis xyz="0 0 1"/>
+        <limit effort="${wheel_effort}" velocity="${wheel_velocity}"/>
+        <dynamics damping="${wheel_damping}" friction="${wheel_friction}"/>
     </joint>
     <link name="left_front_wheel">
         <visual>
             <geometry>
-                <cylinder radius="0.0325" length="0.02"/>
+                <cylinder radius="${wheel_radius}" length="${wheel_length}"/>
             </geometry>
             <material name="blue"/>
@@ -58,8 +47,8 @@
         <collision>
             <geometry>
-                <cylinder radius="0.0325" length="0.02"/>
+                <cylinder radius="${wheel_radius}" length="${wheel_length}"/>
             </geometry>
         </collision>
-        <xacro:inertial_cylinder mass="0.0375" length="0.02" radius="0.0325">
+        <xacro:inertial_cylinder mass="${wheel_mass}" length="${wheel_length}" radius="${wheel_radius}">
             <origin xyz="0 0 0" rpy="0 0 0"/>
         </xacro:inertial_cylinder>
@@ -69,11 +58,13 @@
         <parent link="base_link"/>
         <child link="right_front_wheel"/>
-        <origin xyz="0.0676 -0.0566 0" rpy="${pi/2} 0 0"/>
-        <axis xyz="0 0 -1"/>
+        <origin xyz="${wheel_x_offset} -${wheel_y_offset} ${wheel_z_offset}" rpy="-${pi/2} 0 0"/>
+        <axis xyz="0 0 1"/>
+        <limit effort="${wheel_effort}" velocity="${wheel_velocity}"/>
+        <dynamics damping="${wheel_damping}" friction="${wheel_friction}"/>
     </joint>
     <link name="right_front_wheel">
         <visual>
             <geometry>
-                <cylinder radius="0.0325" length="0.02"/>
+                <cylinder radius="${wheel_radius}" length="${wheel_length}"/>
             </geometry>
             <material name="blue"/>
@@ -81,8 +72,8 @@
         <collision>
             <geometry>
-                <cylinder radius="0.0325" length="0.02"/>
+                <cylinder radius="${wheel_radius}" length="${wheel_length}"/>
             </geometry>
         </collision>
-        <xacro:inertial_cylinder mass="0.0375" length="0.02" radius="0.0325">
+        <xacro:inertial_cylinder mass="${wheel_mass}" length="${wheel_length}" radius="${wheel_radius}">
             <origin xyz="0 0 0" rpy="0 0 0"/>
         </xacro:inertial_cylinder>
@@ -92,11 +83,13 @@
         <parent link="base_link"/>
         <child link="left_rear_wheel"/>
-        <origin xyz="-0.0676 0.0566 0" rpy="-${pi/2} 0 0"/>
+        <origin xyz="-${wheel_x_offset} ${wheel_y_offset} ${wheel_z_offset}" rpy="-${pi/2} 0 0"/>
         <axis xyz="0 0 1"/>
+        <limit effort="${wheel_effort}" velocity="${wheel_velocity}"/>
+        <dynamics damping="${wheel_damping}" friction="${wheel_friction}"/>
     </joint>
     <link name="left_rear_wheel">
         <visual>
             <geometry>
-                <cylinder radius="0.0325" length="0.02"/>
+                <cylinder radius="${wheel_radius}" length="${wheel_length}"/>
             </geometry>
             <material name="black"/>
@@ -104,8 +97,8 @@
         <collision>
             <geometry>
-                <cylinder radius="0.0325" length="0.02"/>
+                <cylinder radius="${wheel_radius}" length="${wheel_length}"/>
             </geometry>
         </collision>
-        <xacro:inertial_cylinder mass="0.0375" length="0.02" radius="0.0325">
+        <xacro:inertial_cylinder mass="${wheel_mass}" length="${wheel_length}" radius="${wheel_radius}">
             <origin xyz="0 0 0" rpy="0 0 0"/>
         </xacro:inertial_cylinder>
@@ -115,11 +108,13 @@
         <parent link="base_link"/>
         <child link="right_rear_wheel"/>
-        <origin xyz="-0.0676 -0.0566 0" rpy="${pi/2} 0 0"/>
-        <axis xyz="0 0 -1"/>
+        <origin xyz="-${wheel_x_offset} -${wheel_y_offset} ${wheel_z_offset}" rpy="-${pi/2} 0 0"/>
+        <axis xyz="0 0 1"/>
+        <limit effort="${wheel_effort}" velocity="${wheel_velocity}"/>
+        <dynamics damping="${wheel_damping}" friction="${wheel_friction}"/>
     </joint>
     <link name="right_rear_wheel">
         <visual>
             <geometry>
-                <cylinder radius="0.0325" length="0.02"/>
+                <cylinder radius="${wheel_radius}" length="${wheel_length}"/>
             </geometry>
             <material name="black"/>
@@ -127,23 +122,36 @@
         <collision>
             <geometry>
-                <cylinder radius="0.0325" length="0.02"/>
+                <cylinder radius="${wheel_radius}" length="${wheel_length}"/>
             </geometry>
         </collision>
-        <xacro:inertial_cylinder mass="0.0375" length="0.02" radius="0.0325">
+        <xacro:inertial_cylinder mass="${wheel_mass}" length="${wheel_length}" radius="${wheel_radius}">
             <origin xyz="0 0 0" rpy="0 0 0"/>
         </xacro:inertial_cylinder>
     </link>
     <!-- GAZEBO MATERIALS -->
+    <gazebo reference="chassis">
+        <material>Gazebo/White</material>
+        <mu1>1.0</mu1>
+        <mu2>1.0</mu2>
+    </gazebo>
     <gazebo reference="left_front_wheel">
         <material>Gazebo/Blue</material>
+        <mu1>1.0</mu1>
+        <mu2>1.0</mu2>
     </gazebo>
     <gazebo reference="right_front_wheel">
         <material>Gazebo/Blue</material>
+        <mu1>1.0</mu1>
+        <mu2>1.0</mu2>
     </gazebo>
     <gazebo reference="left_rear_wheel">
         <material>Gazebo/Black</material>
+        <mu1>1.0</mu1>
+        <mu2>1.0</mu2>
     </gazebo>
     <gazebo reference="right_rear_wheel">
         <material>Gazebo/Black</material>
+        <mu1>1.0</mu1>
+        <mu2>1.0</mu2>
     </gazebo>
 </robot>
