Commit message: Fixed camera orientation

File: description/depth_camera.xacro (robot description, xacro)
@@ -26,5 +26,5 @@
         <parent link="camera_link"/>
         <child link="camera_link_optical"/>
-        <origin xyz="0 0 0" rpy="${-pi/2} 0 ${-pi/2}"/>
+        <origin xyz="0 0 0" rpy="0 ${-pi/2} ${-pi/2}"/>
     </joint>
     <link name="camera_link_optical"></link>

Commit message: Updated camera orientation

File: description/depth_camera.xacro (robot description, xacro)
@@ -26,5 +26,5 @@
         <parent link="camera_link"/>
         <child link="camera_link_optical"/>
-        <origin xyz="0 0 0" rpy="0 ${-pi/2} ${-pi/2}"/>
+        <origin xyz="0 0 0" rpy="0 0 0"/>
     </joint>
     <link name="camera_link_optical"></link>

Commit message: Updated camera orientation

File: description/depth_camera.xacro (robot description, xacro)
@@ -26,5 +26,5 @@
         <parent link="camera_link"/>
         <child link="camera_link_optical"/>
-        <origin xyz="0 0 0" rpy="0 0 0"/>
+        <origin xyz="0 0 0" rpy="-${pi/2} 0 0"/>
     </joint>
     <link name="camera_link_optical"></link>

Commit message: Updated camera orientation in rviz2

File: description/depth_camera.xacro (robot description, xacro)
@@ -26,10 +26,10 @@
         <parent link="camera_link"/>
         <child link="camera_link_optical"/>
-        <origin xyz="0 0 0" rpy="-${pi/2} 0 0"/>
+        <origin xyz="0 0 0" rpy="0 0 0"/>
     </joint>
     <link name="camera_link_optical"></link>
     <gazebo reference="camera_link">
         <sensor name="camera" type="depth">
-            <pose> 0 0 0 0 0 0 </pose>
+            <pose> 0 0 0 -${pi/2} 0 0 </pose>
                 <visualize>true</visualize>
                 <update_rate>10</update_rate>

Commit message: Fixed camera orientation

File: description/depth_camera.xacro (robot description, xacro)
@@ -26,10 +26,10 @@
         <parent link="camera_link"/>
         <child link="camera_link_optical"/>
-        <origin xyz="0 0 0" rpy="0 0 0"/>
+        <origin xyz="0 0 0" rpy="${-pi/2} ${-pi/2}0"/>
     </joint>
     <link name="camera_link_optical"></link>
     <gazebo reference="camera_link">
         <sensor name="camera" type="depth">
-            <pose> 0 0 0 -${pi/2} 0 0 </pose>
+            <pose> 0 0 0 0 0 0 </pose>
                 <visualize>true</visualize>
                 <update_rate>10</update_rate>

Commit message: Corrected camera orientation

File: description/depth_camera.xacro (robot description, xacro)
@@ -26,5 +26,5 @@
         <parent link="camera_link"/>
         <child link="camera_link_optical"/>
-        <origin xyz="0 0 0" rpy="${-pi/2} ${-pi/2}0"/>
+        <origin xyz="0 0 0" rpy="0 0 0"/>
     </joint>
     <link name="camera_link_optical"></link>

Commit message: fixed camera orientation

File: description/depth_camera.xacro (robot description, xacro)
@@ -26,5 +26,5 @@
         <parent link="camera_link"/>
         <child link="camera_link_optical"/>
-        <origin xyz="0 0 0" rpy="0 0 0"/>
+        <origin xyz="0 0 0" rpy="-${pi/2} 0 -${pi/2}"/>
     </joint>
     <link name="camera_link_optical"></link>

Commit message: fixed camera orientation, try #2

File: description/depth_camera.xacro (robot description, xacro)
@@ -5,5 +5,5 @@
         <parent link="chassis"/>
         <child link="camera_link"/>
-        <origin xyz="${camera_origin_x} ${camera_origin_y} ${camera_origin_z}" rpy="0 0 0"/>
+        <origin xyz="${camera_origin_x} ${camera_origin_y} ${camera_origin_z}" rpy="0 ${pi/2} 0"/>
     </joint>
     <link name="camera_link">

Commit message: fixed camera orientation, try #3

File: description/depth_camera.xacro (robot description, xacro)
@@ -5,5 +5,5 @@
         <parent link="chassis"/>
         <child link="camera_link"/>
-        <origin xyz="${camera_origin_x} ${camera_origin_y} ${camera_origin_z}" rpy="0 ${pi/2} 0"/>
+        <origin xyz="${camera_origin_x} ${camera_origin_y} ${camera_origin_z}" rpy="-${pi/2} ${pi/2} 0"/>
     </joint>
     <link name="camera_link">

Commit message: fixed camera orientation, try #4

File: description/depth_camera.xacro (robot description, xacro)
@@ -5,5 +5,5 @@
         <parent link="chassis"/>
         <child link="camera_link"/>
-        <origin xyz="${camera_origin_x} ${camera_origin_y} ${camera_origin_z}" rpy="-${pi/2} ${pi/2} 0"/>
+        <origin xyz="${camera_origin_x} ${camera_origin_y} ${camera_origin_z}" rpy="0 ${pi/2} -${pi/2}"/>
     </joint>
     <link name="camera_link">

Commit message: fixed camera orientation, try #5

File: description/depth_camera.xacro (robot description, xacro)
@@ -5,5 +5,5 @@
         <parent link="chassis"/>
         <child link="camera_link"/>
-        <origin xyz="${camera_origin_x} ${camera_origin_y} ${camera_origin_z}" rpy="0 ${pi/2} -${pi/2}"/>
+        <origin xyz="${camera_origin_x} ${camera_origin_y} ${camera_origin_z}" rpy="${pi/2} ${pi/2} 0"/>
     </joint>
     <link name="camera_link">

Commit message: fixed camera orientation, try #6

File: description/depth_camera.xacro (robot description, xacro)
@@ -5,5 +5,5 @@
         <parent link="chassis"/>
         <child link="camera_link"/>
-        <origin xyz="${camera_origin_x} ${camera_origin_y} ${camera_origin_z}" rpy="${pi/2} ${pi/2} 0"/>
+        <origin xyz="${camera_origin_x} ${camera_origin_y} ${camera_origin_z}" rpy="${pi/2} 0 -${pi/2}"/>
     </joint>
     <link name="camera_link">

Commit message: fixed camera orientation, try #7

File: description/depth_camera.xacro (robot description, xacro)
@@ -26,5 +26,5 @@
         <parent link="camera_link"/>
         <child link="camera_link_optical"/>
-        <origin xyz="0 0 0" rpy="-${pi/2} 0 -${pi/2}"/>
+        <origin xyz="0 0 0" rpy="-${pi/2} 0 0"/>
     </joint>
     <link name="camera_link_optical"></link>

Commit message: fixed camera orientation, try #8

File: description/depth_camera.xacro (robot description, xacro)
@@ -5,5 +5,5 @@
         <parent link="chassis"/>
         <child link="camera_link"/>
-        <origin xyz="${camera_origin_x} ${camera_origin_y} ${camera_origin_z}" rpy="${pi/2} 0 -${pi/2}"/>
+        <origin xyz="${camera_origin_x} ${camera_origin_y} ${camera_origin_z}" rpy="0 ${pi/2} ${pi/2}"/>
     </joint>
     <link name="camera_link">
@@ -26,5 +26,5 @@
         <parent link="camera_link"/>
         <child link="camera_link_optical"/>
-        <origin xyz="0 0 0" rpy="-${pi/2} 0 0"/>
+        <origin xyz="0 0 0" rpy="-${pi/2} 0 -${pi/2}"/>
     </joint>
     <link name="camera_link_optical"></link>

Commit message: fixed camera orientation, try #9

File: description/depth_camera.xacro (robot description, xacro)
@@ -5,5 +5,5 @@
         <parent link="chassis"/>
         <child link="camera_link"/>
-        <origin xyz="${camera_origin_x} ${camera_origin_y} ${camera_origin_z}" rpy="0 ${pi/2} ${pi/2}"/>
+        <origin xyz="${camera_origin_x} ${camera_origin_y} ${camera_origin_z}" rpy="0 0 0"/>
     </joint>
     <link name="camera_link">
@@ -26,5 +26,5 @@
         <parent link="camera_link"/>
         <child link="camera_link_optical"/>
-        <origin xyz="0 0 0" rpy="-${pi/2} 0 -${pi/2}"/>
+        <origin xyz="0 0 0" rpy="0 0 0"/>
     </joint>
     <link name="camera_link_optical"></link>

Commit message: fixed camera orientation, try #12

File: description/depth_camera.xacro (robot description, xacro)
@@ -5,5 +5,5 @@
         <parent link="chassis"/>
         <child link="camera_link"/>
-        <origin xyz="${camera_origin_x} ${camera_origin_y} ${camera_origin_z}" rpy="0 ${pi/2} 0"/>
+        <origin xyz="${camera_origin_x} ${camera_origin_y} ${camera_origin_z}" rpy="${pi/2} ${pi/2} 0"/>
     </joint>
     <link name="camera_link">

Commit message: fixed camera orientation, try #13

File: description/depth_camera.xacro (robot description, xacro)
@@ -5,5 +5,5 @@
         <parent link="chassis"/>
         <child link="camera_link"/>
-        <origin xyz="${camera_origin_x} ${camera_origin_y} ${camera_origin_z}" rpy="${pi/2} ${pi/2} 0"/>
+        <origin xyz="${camera_origin_x} ${camera_origin_y} ${camera_origin_z}" rpy="0 ${pi/2} ${pi/2}"/>
     </joint>
     <link name="camera_link">

Commit message: fixed camera orientation, try #14

File: description/depth_camera.xacro (robot description, xacro)
@@ -5,5 +5,5 @@
         <parent link="chassis"/>
         <child link="camera_link"/>
-        <origin xyz="${camera_origin_x} ${camera_origin_y} ${camera_origin_z}" rpy="0 ${pi/2} ${pi/2}"/>
+        <origin xyz="${camera_origin_x} ${camera_origin_y} ${camera_origin_z}" rpy="${pi/2} ${pi/2} ${pi/2}"/>
     </joint>
     <link name="camera_link">

Commit message: fixed camera orientation, try #15

File: description/depth_camera.xacro (robot description, xacro)
@@ -5,5 +5,5 @@
         <parent link="chassis"/>
         <child link="camera_link"/>
-        <origin xyz="${camera_origin_x} ${camera_origin_y} ${camera_origin_z}" rpy="${pi/2} ${pi/2} ${pi/2}"/>
+        <origin xyz="${camera_origin_x} ${camera_origin_y} ${camera_origin_z}" rpy="${pi/2} ${pi/2} -${pi/2}"/>
     </joint>
     <link name="camera_link">

Commit message: fixed camera orientation, try #16

File: description/depth_camera.xacro (robot description, xacro)
@@ -5,5 +5,5 @@
         <parent link="chassis"/>
         <child link="camera_link"/>
-        <origin xyz="${camera_origin_x} ${camera_origin_y} ${camera_origin_z}" rpy="${pi/2} ${pi/2} -${pi/2}"/>
+        <origin xyz="${camera_origin_x} ${camera_origin_y} ${camera_origin_z}" rpy="-${pi/2} ${pi/2} ${pi/2}"/>
     </joint>
     <link name="camera_link">

Commit message: fixed camera orientation, try #17

File: description/depth_camera.xacro (robot description, xacro)
@@ -5,5 +5,5 @@
         <parent link="chassis"/>
         <child link="camera_link"/>
-        <origin xyz="${camera_origin_x} ${camera_origin_y} ${camera_origin_z}" rpy="-${pi/2} ${pi/2} ${pi/2}"/>
+        <origin xyz="${camera_origin_x} ${camera_origin_y} ${camera_origin_z}" rpy="${pi/2} -${pi/2} ${pi/2}"/>
     </joint>
     <link name="camera_link">

Commit message: fixed camera orientation, try #18

File: description/depth_camera.xacro (robot description, xacro)
@@ -5,5 +5,5 @@
         <parent link="chassis"/>
         <child link="camera_link"/>
-        <origin xyz="${camera_origin_x} ${camera_origin_y} ${camera_origin_z}" rpy="${pi/2} -${pi/2} ${pi/2}"/>
+        <origin xyz="${camera_origin_x} ${camera_origin_y} ${camera_origin_z}" rpy="${pi/2} 0 ${pi/2}"/>
     </joint>
     <link name="camera_link">
