Commit message: Corrected lidar orientation

File: description/lidar.xacro (robot description, xacro)
@@ -4,8 +4,8 @@
     <joint name="laser_joint" type="fixed">
         <parent link="chassis"/>
-        <child link="laser_frame"/>
-        <origin xyz="${lidar_origin_x} ${lidar_origin_y} ${lidar_origin_z}" rpy="0 0 0"/>
+        <child link="base_laser"/>
+        <origin xyz="${lidar_origin_x} ${lidar_origin_y} ${lidar_origin_z}" rpy="0 ${-pi/2} 0"/>
     </joint>
-    <link name="laser_frame">
+    <link name="base_laser">
         <visual>
             <geometry>
@@ -23,5 +23,5 @@
         </xacro:inertial_cylinder>
     </link>
-    <gazebo reference="laser_frame">
+    <gazebo reference="base_laser">
         <sensor name="laser" type="ray">
             <pose> 0 0 0 0 0 0 </pose>

Commit message: Corrected lidar orientation

File: description/lidar.xacro (robot description, xacro)
@@ -5,5 +5,5 @@
         <parent link="chassis"/>
         <child link="base_laser"/>
-        <origin xyz="${lidar_origin_x} ${lidar_origin_y} ${lidar_origin_z}" rpy="0 ${-pi/2} 0"/>
+        <origin xyz="${lidar_origin_x} ${lidar_origin_y} ${lidar_origin_z}" rpy="0 0 ${-pi/2}"/>
     </joint>
     <link name="base_laser">

Commit message: Corrected lidar orientation

File: description/lidar.xacro (robot description, xacro)
@@ -5,5 +5,5 @@
         <parent link="chassis"/>
         <child link="base_laser"/>
-        <origin xyz="${lidar_origin_x} ${lidar_origin_y} ${lidar_origin_z}" rpy="0 0 ${-pi/2}"/>
+        <origin xyz="${lidar_origin_x} ${lidar_origin_y} ${lidar_origin_z}" rpy="0 0 ${pi/2}"/>
     </joint>
     <link name="base_laser">

Commit message: Corrected lidar orientation

File: description/lidar.xacro (robot description, xacro)
@@ -5,5 +5,5 @@
         <parent link="chassis"/>
         <child link="base_laser"/>
-        <origin xyz="${lidar_origin_x} ${lidar_origin_y} ${lidar_origin_z}" rpy="0 0 ${pi/2}"/>
+        <origin xyz="${lidar_origin_x} ${lidar_origin_y} ${lidar_origin_z}" rpy="0 0 ${-pi/2}"/>
     </joint>
     <link name="base_laser">

Commit message: Corrected lidar orientation

File: description/lidar.xacro (robot description, xacro)
@@ -5,5 +5,5 @@
         <parent link="chassis"/>
         <child link="base_laser"/>
-        <origin xyz="${lidar_origin_x} ${lidar_origin_y} ${lidar_origin_z}" rpy="0 0 ${-pi/2}"/>
+        <origin xyz="${lidar_origin_x} ${lidar_origin_y} ${lidar_origin_z}" rpy="0 0 ${pi}"/>
     </joint>
     <link name="base_laser">

Commit message: Corrected lidar orientation

File: description/lidar.xacro (robot description, xacro)
@@ -5,5 +5,5 @@
         <parent link="chassis"/>
         <child link="base_laser"/>
-        <origin xyz="${lidar_origin_x} ${lidar_origin_y} ${lidar_origin_z}" rpy="0 0 ${pi}"/>
+        <origin xyz="${lidar_origin_x} ${lidar_origin_y} ${lidar_origin_z}" rpy="0 0 0"/>
     </joint>
     <link name="base_laser">

Commit message: Corrected lidar orientation

File: description/lidar.xacro (robot description, xacro)
@@ -5,5 +5,5 @@
         <parent link="chassis"/>
         <child link="base_laser"/>
-        <origin xyz="${lidar_origin_x} ${lidar_origin_y} ${lidar_origin_z}" rpy="0 0 0"/>
+        <origin xyz="${lidar_origin_x} ${lidar_origin_y} ${lidar_origin_z}" rpy="0 0 ${pi/2}"/>
     </joint>
     <link name="base_laser">

Commit message: fixed lidar orientation, try #1

File: description/lidar.xacro (robot description, xacro)
@@ -5,5 +5,5 @@
         <parent link="chassis"/>
         <child link="base_laser"/>
-        <origin xyz="${lidar_origin_x} ${lidar_origin_y} ${lidar_origin_z}" rpy="0 0 ${pi/2}"/>
+        <origin xyz="${lidar_origin_x} ${lidar_origin_y} ${lidar_origin_z}" rpy="0 0 -${pi/2}"/>
     </joint>
     <link name="base_laser">

Commit message: fixed lidar orientation, try #2

File: description/lidar.xacro (robot description, xacro)
@@ -5,5 +5,5 @@
         <parent link="chassis"/>
         <child link="base_laser"/>
-        <origin xyz="${lidar_origin_x} ${lidar_origin_y} ${lidar_origin_z}" rpy="0 0 -${pi/2}"/>
+        <origin xyz="${lidar_origin_x} ${lidar_origin_y} ${lidar_origin_z}" rpy="0 0 0"/>
     </joint>
     <link name="base_laser">

Commit message: fixed lidar orientation, try #4

File: description/lidar.xacro (robot description, xacro)
@@ -5,5 +5,5 @@
         <parent link="chassis"/>
         <child link="base_laser"/>
-        <origin xyz="${lidar_origin_x} ${lidar_origin_y} ${lidar_origin_z}" rpy="0 0 ${pi/2}"/>
+        <origin xyz="${lidar_origin_x} ${lidar_origin_y} ${lidar_origin_z}" rpy="${pi/2} 0 ${pi/2}"/>
     </joint>
     <link name="base_laser">

Commit message: fixed lidar orientation, try #5

File: description/lidar.xacro (robot description, xacro)
@@ -5,5 +5,5 @@
         <parent link="chassis"/>
         <child link="base_laser"/>
-        <origin xyz="${lidar_origin_x} ${lidar_origin_y} ${lidar_origin_z}" rpy="${pi/2} 0 ${pi/2}"/>
+        <origin xyz="${lidar_origin_x} ${lidar_origin_y} ${lidar_origin_z}" rpy="0 0 -${pi/2}"/>
     </joint>
     <link name="base_laser">

Commit message: fixed lidar orientation, try #9

File: description/lidar.xacro (robot description, xacro)
@@ -5,5 +5,5 @@
         <parent link="chassis"/>
         <child link="base_laser"/>
-        <origin xyz="${lidar_origin_x} ${lidar_origin_y} ${lidar_origin_z}" rpy="0 0 -${pi/2}"/>
+        <origin xyz="${lidar_origin_x} ${lidar_origin_y} ${lidar_origin_z}" rpy="0 0 ${pi/2}"/>
     </joint>
     <link name="base_laser">

Commit message: fixed lidar orientation, try #10

File: description/lidar.xacro (robot description, xacro)
@@ -5,5 +5,5 @@
         <parent link="chassis"/>
         <child link="base_laser"/>
-        <origin xyz="${lidar_origin_x} ${lidar_origin_y} ${lidar_origin_z}" rpy="0 0 ${pi/2}"/>
+        <origin xyz="${lidar_origin_x} ${lidar_origin_y} ${lidar_origin_z}" rpy="0 ${pi/2} 0"/>
     </joint>
     <link name="base_laser">

Commit message: fixed lidar orientation, try #11

File: description/lidar.xacro (robot description, xacro)
@@ -5,5 +5,5 @@
         <parent link="chassis"/>
         <child link="base_laser"/>
-        <origin xyz="${lidar_origin_x} ${lidar_origin_y} ${lidar_origin_z}" rpy="0 ${pi/2} 0"/>
+        <origin xyz="${lidar_origin_x} ${lidar_origin_y} ${lidar_origin_z}" rpy="0 ${pi/2} -${pi/2}"/>
     </joint>
     <link name="base_laser">

Commit message: fixed lidar orientation, try #12

File: description/lidar.xacro (robot description, xacro)
@@ -5,5 +5,5 @@
         <parent link="chassis"/>
         <child link="base_laser"/>
-        <origin xyz="${lidar_origin_x} ${lidar_origin_y} ${lidar_origin_z}" rpy="0 ${pi/2} -${pi/2}"/>
+        <origin xyz="${lidar_origin_x} ${lidar_origin_y} ${lidar_origin_z}" rpy="0 0-${pi/2}"/>
     </joint>
     <link name="base_laser">
@@ -48,5 +48,5 @@
                     </ros>
                     <output_type>sensor_msgs/LaserScan</output_type>
-                    <frame_name>laser_frame</frame_name>
+                    <frame_name>base_laser</frame_name>
                 </plugin>
         </sensor>

Commit message: fixed lidar orientation, try #12

File: description/lidar.xacro (robot description, xacro)
@@ -5,5 +5,5 @@
         <parent link="chassis"/>
         <child link="base_laser"/>
-        <origin xyz="${lidar_origin_x} ${lidar_origin_y} ${lidar_origin_z}" rpy="0 0-${pi/2}"/>
+        <origin xyz="${lidar_origin_x} ${lidar_origin_y} ${lidar_origin_z}" rpy="0 0 -${pi/2}"/>
     </joint>
     <link name="base_laser">

Commit message: fixed lidar orientation, try #15

File: description/lidar.xacro (robot description, xacro)
@@ -5,5 +5,5 @@
         <parent link="chassis"/>
         <child link="base_laser"/>
-        <origin xyz="${lidar_origin_x} ${lidar_origin_y} ${lidar_origin_z}" rpy="0 0 ${pi/2}"/>
+        <origin xyz="${lidar_origin_x} ${lidar_origin_y} ${lidar_origin_z}" rpy="${pi} 0 -${pi/2}"/>
     </joint>
     <link name="base_laser">

Commit message: fixed lidar orientation, try #16

File: description/lidar.xacro (robot description, xacro)
@@ -5,5 +5,5 @@
         <parent link="chassis"/>
         <child link="base_laser"/>
-        <origin xyz="${lidar_origin_x} ${lidar_origin_y} ${lidar_origin_z}" rpy="${pi} 0 -${pi/2}"/>
+        <origin xyz="${lidar_origin_x} ${lidar_origin_y} ${lidar_origin_z}" rpy="${pi} 0 ${pi/2}"/>
     </joint>
     <link name="base_laser">

Commit message: fixed lidar orientation, try #17

File: description/lidar.xacro (robot description, xacro)
@@ -5,5 +5,5 @@
         <parent link="chassis"/>
         <child link="base_laser"/>
-        <origin xyz="${lidar_origin_x} ${lidar_origin_y} ${lidar_origin_z}" rpy="${pi} 0 ${pi/2}"/>
+        <origin xyz="${lidar_origin_x} ${lidar_origin_y} ${lidar_origin_z}" rpy="0 0 -${pi/2}"/>
     </joint>
     <link name="base_laser">
@@ -48,5 +48,5 @@
                     </ros>
                     <output_type>sensor_msgs/LaserScan</output_type>
-                    <frame_name>base_laser</frame_name>
+                    <frame_name>laser_frame</frame_name>
                 </plugin>
         </sensor>
